Commit message: update

File: ros-env/catkin_ws/src/urdf_store/urdf/hc10/hc10dt.urdf.xacro (robot description, xacro)
@@ -92,5 +92,5 @@
         <geometry>
           <mesh filename="package://motoman_hc10_support/meshes/hc10dt/collision/link_6_t.stl"/>
-       </geometry>
+        </geometry>
       </collision>
     </link>
@@ -100,14 +100,14 @@
       <visual>
         <geometry>
-          <mesh filename="package://urdf_store/urdf/hand/base_hand_pitch_linear_2dof_nozzleguard.stl" />
+          <mesh filename="package://urdf_store/urdf/hand/l1_hand_for_hc10.stl" />
         </geometry>
         <origin rpy="0.0 0.0 0.0" xyz="0.0 0.0 0.0" />
-        <material name="Gray">
-          <color rgba="0.5 0.5 0.5 1.0" />
+        <material name="Grey">
+          <color rgba="0.5 0.5 0.5 1.0"/>
         </material>
       </visual>
       <collision>
         <geometry>
-          <mesh filename="package://urdf_store/urdf/hand/base_hand_pitch_linear_2dof_nozzleguard.stl" />
+          <mesh filename="package://urdf_store/urdf/hand/l1_hand_for_hc10.stl" />
         </geometry>
         <origin rpy="0.0 0.0 0.0" xyz="0.0 0.0 0.0" />
@@ -141,7 +141,7 @@
       <parent link="${prefix}link_2_l"/>
       <child link="${prefix}link_3_u"/>
-      <origin xyz="0 0 0.700" rpy="0 0 0" />
+      <origin xyz="0 0 0.700" rpy="0 ${-pi/2} 0" />
       <axis xyz="0 -1 0" />
-      <limit lower="${radians(-5)}" upper="${radians(355)}" effort="141.12" velocity="${radians(180)}"/>
+      <limit lower="${radians(-95)}" upper="${radians(265)}" effort="141.12" velocity="${radians(180)}"/>
     </joint>
     <joint name="${prefix}joint_4_r" type="revolute">
@@ -164,8 +164,8 @@
       <origin xyz="0 0 0" rpy="0 0 0" />
       <axis xyz="0 0 1" />
-      <limit lower="${radians(-180)}" upper="${radians(180)}" effort="31.36" velocity="${radians(250)}"/>
+      <limit lower="${radians(-210)}" upper="${radians(210)}" effort="31.36" velocity="${radians(250)}"/>
     </joint>
     <joint name="${prefix}joint_6_t-tool0" type="fixed">
-      <origin xyz="0 0 -0.170" rpy="${pi} 0 0"/>
+      <origin xyz="0 0 -0.170" rpy="${pi} 0 ${-pi/2}"/>
       <parent link="${prefix}link_6_t"/>
       <child link="${prefix}tool0"/>
@@ -174,11 +174,12 @@
     <joint name="${prefix}ee_fixed_joint" type="fixed">
       <parent link="${prefix}tool0" />
-      <child link="${prefix}ee_link" />
-      <origin xyz="0.0 -0.1 0.2665" rpy="0.0 0.0 0.0" />
+      <child link = "${prefix}ee_link" />
+      <!-- <origin xyz="0.0 -0.1 0.3115" rpy="0.0 0.0 0.0" /> -->
+      <origin xyz="0.0 -0.253 0.496" rpy="0.0 0.0 0.0" />
     </joint>
     <joint name="${prefix}ee_forcesensor_joint" type="fixed">
       <parent link="${prefix}tool0" />
-      <child link="${prefix}ee_forcesensor" />
-      <origin xyz="0.0 -0.1 0.0573" rpy="0.0 0.0 ${pi/2}" />
+      <child link = "${prefix}ee_forcesensor" />
+      <origin xyz="0.0 -0.2 0.0573" rpy="0.0 0.0 ${pi/2}" />
     </joint>
     <!-- end of hand joint list -->
@@ -197,5 +198,5 @@
         <geometry>
           <!--
-          <mesh filename="package://ppr_sandbox_botamochi_sandbox/urdf/stand/2022_Yaskawa_robotbaseorigine_lowpolygon.stl" />
+          <mesh filename="package://urdf_store/urdf/stand/2022_Yaskawa_robotbaseorigine_lowpolygon.stl" />
           -->
           <mesh filename="package://urdf_store/urdf/stand/base_and_stand.stl" />
@@ -209,5 +210,5 @@
         <geometry>
           <!--
-          <mesh filename="package://ppr_sandbox_botamochi_sandbox/urdf/stand/2022_Yaskawa_robotbaseorigine_lowpolygon.stl" />
+          <mesh filename="package://urdf_store/urdf/stand/2022_Yaskawa_robotbaseorigine_lowpolygon.stl" />
           -->
           <mesh filename="package://urdf_store/urdf/stand/base_and_stand.stl" />

File: ros-env/catkin_ws/src/urdf_store/urdf/hc10/hc10dt_calib.urdf.xacro (robot description, xacro)
@@ -85,11 +85,11 @@
       <visual>
         <geometry>
-          <mesh filename="package://motoman_hc10_support/meshes/hc10/visual/link_6_t.dae"/>
-        </geometry>
-        <xacro:material_yaskawa_blue/>
-      </visual>
-      <collision>
-        <geometry>
-          <mesh filename="package://motoman_hc10_support/meshes/hc10/collision/link_6_t.stl"/>
+          <mesh filename="package://motoman_hc10_support/meshes/hc10dt/visual/link_6_t.dae"/>
+        </geometry>
+        <xacro:material_yaskawa_blue/>
+      </visual>
+      <collision>
+        <geometry>
+          <mesh filename="package://motoman_hc10_support/meshes/hc10dt/collision/link_6_t.stl"/>
         </geometry>
       </collision>
@@ -100,5 +100,5 @@
       <visual>
         <geometry>
-          <mesh filename="package://ppr_sandbox_botamochi_sandbox/urdf/hand/ensenso_calib_board_for_hc10.stl" />
+          <mesh filename="package://urdf_store/urdf/hand/ensenso_calib_board_for_hc10.stl" />
         </geometry>
         <origin rpy="0.0 0.0 0.0" xyz="0.0 0.0 0.0" />
@@ -109,5 +109,5 @@
       <collision>
         <geometry>
-          <mesh filename="package://ppr_sandbox_botamochi_sandbox/urdf/hand/ensenso_calib_board_for_hc10.stl" />
+          <mesh filename="package://urdf_store/urdf/hand/ensenso_calib_board_for_hc10.stl" />
         </geometry>
         <origin rpy="0.0 0.0 0.0" xyz="0.0 0.0 0.0"/>
@@ -166,5 +166,5 @@
     </joint>
     <joint name="${prefix}joint_6_t-tool0" type="fixed">
-      <origin xyz="0 0 -0.130" rpy="${pi} 0 0"/>
+      <origin xyz="0 0 -0.170" rpy="${pi} 0 ${-pi/2}"/>
       <parent link="${prefix}link_6_t"/>
       <child link="${prefix}tool0"/>
@@ -174,5 +174,5 @@
       <parent link="${prefix}tool0" />
       <child link = "${prefix}ee_link" />
-      <origin xyz="0.0 -0.38 0.02" rpy="0.0 0.0 0.0" />
+      <origin xyz="0.0 -0.381 0.019" rpy="0.0 0.0 0.0" />
     </joint>
     <!-- end of hand joint list -->
@@ -191,7 +191,7 @@
         <geometry>
           <!--
-          <mesh filename="package://ppr_sandbox_botamochi_sandbox/urdf/stand/2022_Yaskawa_robotbaseorigine_lowpolygon.stl" />
+          <mesh filename="package://urdf_store/urdf/stand/2022_Yaskawa_robotbaseorigine_lowpolygon.stl" />
           -->
-          <mesh filename="package://ppr_sandbox_botamochi_sandbox/urdf/stand/base_and_stand.stl" />
+          <mesh filename="package://urdf_store/urdf/stand/base_and_stand.stl" />
         </geometry>
         <material name="LightGrey">
@@ -203,7 +203,7 @@
         <geometry>
           <!--
-          <mesh filename="package://ppr_sandbox_botamochi_sandbox/urdf/stand/2022_Yaskawa_robotbaseorigine_lowpolygon.stl" />
+          <mesh filename="package://urdf_store/urdf/stand/2022_Yaskawa_robotbaseorigine_lowpolygon.stl" />
           -->
-          <mesh filename="package://ppr_sandbox_botamochi_sandbox/urdf/stand/base_and_stand.stl" />
+          <mesh filename="package://urdf_store/urdf/stand/base_and_stand.stl" />
         </geometry>
       </collision>

File: ros-env/catkin_ws/src/urdf_store/urdf/hc10/hc10dt_robot_calib.urdf.xacro (robot description, xacro)
@@ -1,5 +1,5 @@
 <?xml version="1.0" ?>
 <robot name="motoman_hc10dt" xmlns:xacro="http://ros.org/wiki/xacro">
-  <xacro:include filename="$(find ppr_sandbox_botamochi_sandbox)/urdf/hc10/hc10dt_calib.urdf.xacro" />
+  <xacro:include filename="$(find urdf_store)/urdf/hc10/hc10dt_calib.urdf.xacro" />
   <xacro:motoman_hc10dt prefix=""/>
   <link name="world" />

File: ros-env/catkin_ws/src/urdf_store/urdf/ur5/ur5.urdf.xacro (robot description, xacro)
@@ -48,5 +48,5 @@
         <origin xyz="0 0 0" rpy="0 0 ${base_correction}"/>
         <geometry>
-          <mesh filename="package://ppr_sandbox_botamochi_sandbox/urdf/stand/base_and_stand.stl" />
+          <mesh filename="package://urdf_store/urdf/stand/base_and_stand.stl" />
         </geometry>
         <material name="LightGrey">
@@ -57,5 +57,5 @@
         <origin xyz="0 0 0" rpy="0 0 ${base_correction}"/>
         <geometry>
-          <mesh filename="package://ppr_sandbox_botamochi_sandbox/urdf/stand/base_and_stand.stl" />
+          <mesh filename="package://urdf_store/urdf/stand/base_and_stand.stl" />
         </geometry>
       </collision>
@@ -307,5 +307,5 @@
       <visual>
         <geometry>
-          <mesh filename="package://ppr_sandbox_botamochi_sandbox/urdf/hand/base_hand_pitch_linear_2dof_nozzleguard.stl" />
+          <mesh filename="package://urdf_store/urdf/hand/base_hand_pitch_linear_2dof_nozzleguard.stl" />
         </geometry>
         <origin rpy="0.0 0.0 0.0" xyz="0.0 0.0 0.0" />
@@ -316,5 +316,5 @@
       <collision>
         <geometry>
-          <mesh filename="package://ppr_sandbox_botamochi_sandbox/urdf/hand/base_hand_pitch_linear_2dof_nozzleguard.stl" />
+          <mesh filename="package://urdf_store/urdf/hand/base_hand_pitch_linear_2dof_nozzleguard.stl" />
         </geometry>
         <origin rpy="0.0 0.0 0.0" xyz="0.0 0.0 0.0" />

File: ros-env/catkin_ws/src/urdf_store/urdf/ur5/ur5_calib.urdf.xacro (robot description, xacro)
@@ -48,5 +48,5 @@
         <origin xyz="0 0 0" rpy="0 0 ${base_correction}"/>
         <geometry>
-          <mesh filename="package://ppr_sandbox_botamochi_sandbox/urdf/stand/base_and_stand.stl" />
+          <mesh filename="package://urdf_store/urdf/stand/base_and_stand.stl" />
         </geometry>
         <material name="LightGrey">
@@ -57,5 +57,5 @@
         <origin xyz="0 0 0" rpy="0 0 ${base_correction}"/>
         <geometry>
-          <mesh filename="package://ppr_sandbox_botamochi_sandbox/urdf/stand/base_and_stand.stl" />
+          <mesh filename="package://urdf_store/urdf/stand/base_and_stand.stl" />
         </geometry>
       </collision>
@@ -306,5 +306,5 @@
       <visual>
         <geometry>
-          <mesh filename="package://ppr_sandbox_botamochi_sandbox/urdf/hand/ensenso_calib_board_for_ur5.stl" />
+          <mesh filename="package://urdf_store/urdf/hand/ensenso_calib_board_for_ur5.stl" />
         </geometry>
         <origin rpy="0.0 0.0 0.0" xyz="0.0 0.0 0.0" />
@@ -315,5 +315,5 @@
       <collision>
         <geometry>
-          <mesh filename="package://ppr_sandbox_botamochi_sandbox/urdf/hand/ensenso_calib_board_for_ur5.stl" />
+          <mesh filename="package://urdf_store/urdf/hand/ensenso_calib_board_for_ur5.stl" />
         </geometry>
         <origin rpy="0.0 0.0 0.0" xyz="0.0 0.0 0.0"/>

File: ros-env/catkin_ws/src/urdf_store/urdf/ur5/ur5_robot.urdf.xacro (robot description, xacro)
@@ -6,7 +6,7 @@
   <xacro:include filename="$(find ur_description)/urdf/common.gazebo.xacro" />
   <!-- ur5 -->
-  <xacro:include filename="$(find ppr_sandbox_botamochi_sandbox)/urdf/ur5/ur5.urdf.xacro" />
+  <xacro:include filename="$(find urdf_store)/urdf/ur5/ur5.urdf.xacro" />
   <!-- arm 20200616 (Avoiding tray entry at the wrist)-->
-  <!--xacro:arg name="kinematics_config" default="$(find ppr_sandbox_botamochi_sandbox)/config/ur5/kinematics_default.yaml"/>
+  <!--xacro:arg name="kinematics_config" default="$(find urdf_store)/config/ur5/kinematics_default.yaml"/>
   <xacro:ur5_robot prefix="" joint_limited="true"
     shoulder_pan_lower_limit="-1.5708" shoulder_pan_upper_limit="1.5708"
@@ -20,5 +20,5 @@
   /-->
   <!-- arm 20200604 (setting up for no collision) -->
-  <xacro:arg name="kinematics_config" default="$(find ppr_sandbox_botamochi_sandbox)/config/ur5/kinematics_default.yaml"/>
+  <xacro:arg name="kinematics_config" default="$(find urdf_store)/config/ur5/kinematics_default.yaml"/>
   <xacro:ur5_robot prefix="" joint_limited="true"
     shoulder_pan_lower_limit="${-0.5 * pi}" shoulder_pan_upper_limit="${0.5833 * pi}"
@@ -38,7 +38,7 @@
   </joint>
   <ppr_tools default="mx35_x1">
-    <xacro:include filename="$(find ppr_sandbox_botamochi_sandbox)/urdf/hand/tool/pigrip25_x2.urdf.xacro" />
-    <xacro:include filename="$(find ppr_sandbox_botamochi_sandbox)/urdf/hand/tool/mx35_x1.urdf.xacro" />
-    <xacro:include filename="$(find ppr_sandbox_botamochi_sandbox)/urdf/hand/tool/pisoftgrip.urdf.xacro" />
+    <xacro:include filename="$(find urdf_store)/urdf/hand/tool/pigrip25_x2.urdf.xacro" />
+    <xacro:include filename="$(find urdf_store)/urdf/hand/tool/mx35_x1.urdf.xacro" />
+    <xacro:include filename="$(find urdf_store)/urdf/hand/tool/pisoftgrip.urdf.xacro" />
   </ppr_tools>
 </robot>

File: ros-env/catkin_ws/src/urdf_store/urdf/ur5/ur5_robot_calib.urdf.xacro (robot description, xacro)
@@ -6,7 +6,7 @@
   <xacro:include filename="$(find ur_description)/urdf/common.gazebo.xacro" />
   <!-- ur5 -->
-  <xacro:include filename="$(find ppr_sandbox_botamochi_sandbox)/urdf/ur5/ur5_calib.urdf.xacro" />
+  <xacro:include filename="$(find urdf_store)/urdf/ur5/ur5_calib.urdf.xacro" />
   <!-- arm -->
-  <xacro:arg name="kinematics_config" default="$(find ppr_sandbox_botamochi_sandbox)/config/ur5/kinematics_default.yaml"/>
+  <xacro:arg name="kinematics_config" default="$(find urdf_store)/config/ur5/kinematics_default.yaml"/>
   <xacro:ur5_robot prefix="" joint_limited="true"
     shoulder_pan_lower_limit="-1.5708" shoulder_pan_upper_limit="1.5708"

File: ros-env/catkin_ws/src/urdf_store/urdf/ur5/ur5e.urdf.xacro (robot description, xacro)
@@ -79,5 +79,5 @@
         <origin xyz="0 0 0" rpy="0 0 ${base_correction}"/>
         <geometry>
-          <mesh filename="package://ppr_sandbox_botamochi_sandbox/urdf/stand/base_and_stand.stl" />
+          <mesh filename="package://urdf_store/urdf/stand/base_and_stand.stl" />
         </geometry>
         <material name="LightGrey">
@@ -88,5 +88,5 @@
         <origin xyz="0 0 0" rpy="0 0 ${base_correction}"/>
         <geometry>
-          <mesh filename="package://ppr_sandbox_botamochi_sandbox/urdf/stand/base_and_stand.stl" />
+          <mesh filename="package://urdf_store/urdf/stand/base_and_stand.stl" />
         </geometry>
       </collision>
@@ -102,5 +102,5 @@
         <origin xyz="0 0 0" rpy="0 0 ${base_correction}"/>
         <geometry>
-          <mesh filename="package://ppr_sandbox_botamochi_sandbox/urdf/stand/base_and_stand.stl" />
+          <mesh filename="package://urdf_store/urdf/stand/base_and_stand.stl" />
         </geometry>
         <material name="LightGrey">
@@ -111,5 +111,5 @@
         <origin xyz="0 0 0" rpy="0 0 ${base_correction}"/>
         <geometry>
-          <mesh filename="package://ppr_sandbox_botamochi_sandbox/urdf/stand/base_and_stand.stl" />
+          <mesh filename="package://urdf_store/urdf/stand/base_and_stand.stl" />
         </geometry>
       </collision>
@@ -361,5 +361,5 @@
       <visual>
         <geometry>
-          <mesh filename="package://ppr_sandbox_botamochi_sandbox/urdf/hand/base_hand_pitch_linear_2dof_nozzleguard.stl" />
+          <mesh filename="package://urdf_store/urdf/hand/base_hand_pitch_linear_2dof_nozzleguard.stl" />
         </geometry>
         <origin rpy="0.0 0.0 0.0" xyz="0.0 0.0 0.0" />
@@ -370,5 +370,5 @@
       <collision>
         <geometry>
-          <mesh filename="package://ppr_sandbox_botamochi_sandbox/urdf/hand/base_hand_pitch_linear_2dof_nozzleguard.stl" />
+          <mesh filename="package://urdf_store/urdf/hand/base_hand_pitch_linear_2dof_nozzleguard.stl" />
         </geometry>
         <origin rpy="0.0 0.0 0.0" xyz="0.0 0.0 0.0" />

File: ros-env/catkin_ws/src/urdf_store/urdf/ur5/ur5e_calib.urdf.xacro (robot description, xacro)
@@ -79,5 +79,5 @@
         <origin xyz="0 0 0" rpy="0 0 ${base_correction}"/>
         <geometry>
-          <mesh filename="package://ppr_sandbox_botamochi_sandbox/urdf/stand/base_and_stand.stl" />
+          <mesh filename="package://urdf_store/urdf/stand/base_and_stand.stl" />
         </geometry>
         <material name="LightGrey">
@@ -88,5 +88,5 @@
         <origin xyz="0 0 0" rpy="0 0 ${base_correction}"/>
         <geometry>
-          <mesh filename="package://ppr_sandbox_botamochi_sandbox/urdf/stand/base_and_stand.stl" />
+          <mesh filename="package://urdf_store/urdf/stand/base_and_stand.stl" />
         </geometry>
       </collision>
@@ -102,5 +102,5 @@
         <origin xyz="0 0 0" rpy="0 0 ${base_correction}"/>
         <geometry>
-          <mesh filename="package://ppr_sandbox_botamochi_sandbox/urdf/stand/base_and_stand.stl" />
+          <mesh filename="package://urdf_store/urdf/stand/base_and_stand.stl" />
         </geometry>
         <material name="LightGrey">
@@ -111,5 +111,5 @@
         <origin xyz="0 0 0" rpy="0 0 ${base_correction}"/>
         <geometry>
-          <mesh filename="package://ppr_sandbox_botamochi_sandbox/urdf/stand/base_and_stand.stl" />
+          <mesh filename="package://urdf_store/urdf/stand/base_and_stand.stl" />
         </geometry>
       </collision>
@@ -367,5 +367,5 @@
       <visual>
         <geometry>
-          <mesh filename="package://ppr_sandbox_botamochi_sandbox/urdf/hand/ensenso_calib_board_for_ur5.stl" />
+          <mesh filename="package://urdf_store/urdf/hand/ensenso_calib_board_for_ur5.stl" />
         </geometry>
         <origin rpy="0.0 0.0 0.0" xyz="0.0 0.0 0.0" />
@@ -376,5 +376,5 @@
       <collision>
         <geometry>
-          <mesh filename="package://ppr_sandbox_botamochi_sandbox/urdf/hand/ensenso_calib_board_for_ur5.stl" />
+          <mesh filename="package://urdf_store/urdf/hand/ensenso_calib_board_for_ur5.stl" />
         </geometry>
         <origin rpy="0.0 0.0 0.0" xyz="0.0 0.0 0.0"/>

File: ros-env/catkin_ws/src/urdf_store/urdf/ur5/ur5e_robot.urdf.xacro (robot description, xacro)
@@ -6,7 +6,7 @@
   <xacro:include filename="$(find ur_description)/urdf/common.gazebo.xacro" />
   <!-- ur5e -->
-  <xacro:include filename="$(find ppr_sandbox_botamochi_sandbox)/urdf/ur5/ur5e.urdf.xacro" />
+  <xacro:include filename="$(find urdf_store)/urdf/ur5/ur5e.urdf.xacro" />
   <!-- arm 20200616 (Avoiding tray entry at the wrist)-->
-  <!--xacro:arg name="kinematics_config" default="$(find ppr_sandbox_botamochi_sandbox)/config/ur5/kinematics_default.yaml"/>
+  <!--xacro:arg name="kinematics_config" default="$(find urdf_store)/config/ur5/kinematics_default.yaml"/>
   <xacro:ur5_robot prefix="" joint_limited="true"
     shoulder_pan_lower_limit="-1.5708" shoulder_pan_upper_limit="1.5708"
@@ -20,5 +20,5 @@
   /-->
   <!-- arm 20210806 (setting up for no collision) -->
-  <xacro:arg name="kinematics_config" default="$(find ppr_sandbox_botamochi_sandbox)/config/ur5e/kinematics_default.yaml"/>
+  <xacro:arg name="kinematics_config" default="$(find urdf_store)/config/ur5e/kinematics_default.yaml"/>
   <xacro:ur5_robot prefix="" joint_limited="true"
     shoulder_pan_lower_limit="-1.5708" shoulder_pan_upper_limit="1.5708"
@@ -38,7 +38,7 @@
   </joint>
   <ppr_tools default="mx35_x1">
-    <xacro:include filename="$(find ppr_sandbox_botamochi_sandbox)/urdf/hand/tool/pigrip25_x2.urdf.xacro" />
-    <xacro:include filename="$(find ppr_sandbox_botamochi_sandbox)/urdf/hand/tool/mx35_x1.urdf.xacro" />
-    <xacro:include filename="$(find ppr_sandbox_botamochi_sandbox)/urdf/hand/tool/pisoftgrip.urdf.xacro" />
+    <xacro:include filename="$(find urdf_store)/urdf/hand/tool/pigrip25_x2.urdf.xacro" />
+    <xacro:include filename="$(find urdf_store)/urdf/hand/tool/mx35_x1.urdf.xacro" />
+    <xacro:include filename="$(find urdf_store)/urdf/hand/tool/pisoftgrip.urdf.xacro" />
   </ppr_tools>
 </robot>

File: ros-env/catkin_ws/src/urdf_store/urdf/ur5/ur5e_robot_calib.urdf.xacro (robot description, xacro)
@@ -6,7 +6,7 @@
   <xacro:include filename="$(find ur_description)/urdf/common.gazebo.xacro" />
   <!-- ur5 -->
-  <xacro:include filename="$(find ppr_sandbox_botamochi_sandbox)/urdf/ur5/ur5e_calib.urdf.xacro" />
+  <xacro:include filename="$(find urdf_store)/urdf/ur5/ur5e_calib.urdf.xacro" />
   <!-- arm -->
-  <xacro:arg name="kinematics_config" default="$(find ppr_sandbox_botamochi_sandbox)/config/ur5e/kinematics_default.yaml"/>
+  <xacro:arg name="kinematics_config" default="$(find urdf_store)/config/ur5e/kinematics_default.yaml"/>
   <xacro:ur5_robot prefix="" joint_limited="true"
     shoulder_pan_lower_limit="-1.5708" shoulder_pan_upper_limit="1.5708"

File: ros-env/catkin_ws/src/urdf_store/urdf/vs087/vs087_calib_vs087-1.urdf (robot description, URDF)
Before this commit: robot vs087, 9 links, 8 joints
Links:
- link ee_link: geometry collision mesh filename=package://urdf_store/urdf/hand/ensenso_calib_board_for_vs08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 scale=1 1 1; visual mesh filename=package://urdf_store/urdf/hand/ensenso_calib_board_for_vs08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 scale=1 1 1

File: ros-env/catkin_ws/src/urdf_store/urdf/vs087/vs087_vs087-1.urdf (robot description, URDF)
Before this commit: robot vs087, 9 links, 8 joints
Links:
- link ee_link: geometry collision mesh filename=package://urdf_store/urdf/hand/15mmx2pad_hand_for_vs087.stl scale=1 1 1; visual mesh filename=package://urdf_store/urdf/hand/15mmx2pad_hand_for_vs087.stl scale=1 1 1
